Commit message: modify the description package for ROS2, add documentation

File: flir_camera_description/urdf/flir_blackfly_s.urdf.xacro (robot description, xacro)
@@ -1,4 +1,4 @@
 <?xml version="1.0"?>
-    <robot xmlns:xacro="http://www.ros.org/wiki/xacro" name="flir_blackflys">
+    <robot xmlns:xacro="http://www.ros.org/wiki/xacro" name="flir_blackfly_s">
     <!--
         camera_{x,y,z,mass} are physical properties of camera collision model
@@ -6,5 +6,5 @@
         hfov, fps, width, height, format, near, and far are simulation
     -->
-    <xacro:macro name="flir_blackflys"
+    <xacro:macro name="flir_blackfly_s"
         params="frame:=camera name:=camera camera_x:=0.047758 camera_y:=0.029 camera_z:=0.029 camera_mass:=0.03
                 lens_r:=0.016 lens_h:=0.04 lens_mass:= 0.05
@@ -18,5 +18,5 @@
             <origin xyz="0 0 0.01425" rpy="0 0 0" />
             <geometry>
-                <mesh filename="package://flir_camera_description/meshes/flir_blackflys.stl"/>
+                <mesh filename="package://flir_camera_description/meshes/flir_blackfly_s.stl"/>
             </geometry>
             <material name="dark_grey" />
